Commit message: add Kd to pitch and yaw controller

File: balegce_gazebo/robot/balegce.gazebo.xacro (robot description, xacro)
@@ -13,10 +13,4 @@
     <!-- <link name="world"/> -->
     <xacro:balegce/>
-    <!-- <joint name="offset" type="floating">
-        <parent link="world"/>
-        <child link="base"/>
-        <origin xyz="0.0 0.0 0.15" rpy="0.0 0.0 0.0"/>
-        <axis xyz="0 0 1"/>
-    </joint> -->
     <xacro:sensor_link/>
     <xacro:sensor_plugins/>

File: balegce_gazebo/robot/balegce_controller.gazebo.xacro (robot description, xacro)
@@ -8,4 +8,8 @@
       </hardware>
       <joint name="joint_body">
+        <command_interface name="position">
+          <param name="min">0.0</param>
+          <param name="max">0.065</param>
+        </command_interface>
         <command_interface name="effort"/>
         <command_interface name="velocity"/>

Commit message: add angular acc cal

File: balegce_gazebo/robot/balegce.gazebo.xacro (robot description, xacro)
@@ -8,5 +8,5 @@
     <xacro:include filename="$(find ${gazebo_pkg})/robot/balegce_sensor.gazebo.xacro"/>
     <xacro:include filename="$(find ${gazebo_pkg})/robot/balegce_controller.gazebo.xacro"/>
-    <xacro:include filename="$(find ${gazebo_pkg})/robot/visual/balegce_ground_truth.xacro"/>
+    <xacro:include filename="$(find ${gazebo_pkg})/robot/balegce_ground_truth.xacro"/>
     <!-- Add manipulator -->
     <xacro:include filename="$(find ${description_pkg})/robot/visual/manipulator.xacro"/>

File: balegce_gazebo/robot/balegce_ground_truth.xacro (robot description, xacro)
@@ -1,21 +1,16 @@
 <?xml version="1.0"?>
-<robot xmlns:controller="http://playerstage.sourceforge.net/gazebo/xmlschema/#controller" name="simple_box">
+<robot xmlns:xacro="http://www.ros.org/wiki/xacro" name="example">
 <!-- ground truth -->
-<xacro:macro name="ground_truth" params="">
-    <gazebo>
-        <controller:ros_p3d name="body_controller" plugin="libros_p3d.so">
+   <xacro:macro name="ground_truth" params="">
+      <gazebo>
+         <plugin filename="libgazebo_ros_p3d.so" name="body_groundtruth_sim">
             <alwaysOn>true</alwaysOn>
             <updateRate>100.0</updateRate>
-            <bodyName>body</bodyName>
-            <topicName>body_pose_ground_truth</topicName>
+            <bodyName>base</bodyName>
+            <topicName>ground_truth/state</topicName>
             <gaussianNoise>0.0</gaussianNoise>
-            <frameName>body</frameName>
-            <interface:position name="body_p3d_position_iface" />
-        </controller:ros_p3d>
-    </gazebo>
-    <gazebo reference="body">
-        <material>Gazebo/Blue</material>
-        <turnGravityOff>false</turnGravityOff>
-    </gazebo>
-</xacro:macro>
+            <frameName>world</frameName>
+         </plugin>
+      </gazebo>
+   </xacro:macro>
 </robot>
