Commit message: add joint state publisher

File: balegce_gazebo/robot/balegce_controller.gazebo.xacro (robot description, xacro)
@@ -7,5 +7,5 @@
         <plugin>gazebo_ros2_control/GazeboSystem</plugin>
       </hardware>
-      <joint name="joint_1">
+      <joint name="joint_wheel">
         <command_interface name="effort"/>
         <command_interface name="velocity"/>

File: balegce_gazebo/robot/balegce_sensor.gazebo.xacro (robot description, xacro)
@@ -3,11 +3,45 @@
     <xacro:macro name="sensor_plugins" params="">
         <!--joint ideal sensor-->
+        <!-- joint_body -->
         <gazebo>
-            <plugin name="joint_state_publisher"
+            <plugin name="joint_body_state_publisher"
                 filename="libgazebo_ros_joint_state_publisher.so">
                 <update_rate>20.0</update_rate>
-                <joint_name>joint_1</joint_name>
+                <joint_name>joint_body</joint_name>
                 <ros>
-                    <remapping>/joint_states:=joint_states</remapping>
+                    <remapping>/joint_states:=joint_body_states</remapping>
+                </ros>
+            </plugin>
+        </gazebo>
+        <!-- joint_wheel -->
+        <gazebo>
+            <plugin name="joint_wheel_state_publisher"
+                filename="libgazebo_ros_joint_state_publisher.so">
+                <update_rate>20.0</update_rate>
+                <joint_name>joint_wheel</joint_name>
+                <ros>
+                    <remapping>/joint_states:=joint_wheel_states</remapping>
+                </ros>
+            </plugin>
+        </gazebo>
+        <!-- joint_propeller_1 -->
+        <gazebo>
+            <plugin name="joint_propeller_1_state_publisher"
+                filename="libgazebo_ros_joint_state_publisher.so">
+                <update_rate>20.0</update_rate>
+                <joint_name>joint_propeller_1</joint_name>
+                <ros>
+                    <remapping>/joint_states:=joint_propeller_1_states</remapping>
+                </ros>
+            </plugin>
+        </gazebo>
+        <!-- joint_propeller_2 -->
+        <gazebo>
+            <plugin name="joint_propeller_2_state_publisher"
+                filename="libgazebo_ros_joint_state_publisher.so">
+                <update_rate>20.0</update_rate>
+                <joint_name>joint_propeller_2</joint_name>
+                <ros>
+                    <remapping>/joint_states:=joint_propeller_2_states</remapping>
                 </ros>
             </plugin>

Commit message: add launch argus for controller gain

File: balegce_gazebo/robot/balegce_controller.gazebo.xacro (robot description, xacro)
@@ -15,4 +15,20 @@
       </joint>
       <joint name="leg">
+        <command_interface name="position"/>
+        <command_interface name="velocity"/>
+        <command_interface name="effort"/>
+        <state_interface name="position"/>
+        <state_interface name="velocity"/>
+        <state_interface name="effort"/>
+      </joint>
+      <joint name="joint_propeller_1">
+        <command_interface name="position"/>
+        <command_interface name="velocity"/>
+        <command_interface name="effort"/>
+        <state_interface name="position"/>
+        <state_interface name="velocity"/>
+        <state_interface name="effort"/>
+      </joint>
+      <joint name="joint_propeller_2">
         <command_interface name="position"/>
         <command_interface name="velocity"/>

Commit message: add threshole and fixed leg

File: balegce_gazebo/robot/balegce_controller.gazebo.xacro (robot description, xacro)
@@ -7,5 +7,5 @@
         <plugin>gazebo_ros2_control/GazeboSystem</plugin>
       </hardware>
-      <joint name="joint_body">
+      <!-- <joint name="joint_body">
         <command_interface name="position">
           <param name="min">0.0</param>
@@ -17,5 +17,5 @@
         <state_interface name="velocity"/>
         <state_interface name="effort"/>
-      </joint>
+      </joint> -->
       <joint name="joint_wheel">
         <command_interface name="effort"/>

Commit message: change joint leg to prismatic

File: balegce_gazebo/robot/balegce_controller.gazebo.xacro (robot description, xacro)
@@ -7,5 +7,5 @@
         <plugin>gazebo_ros2_control/GazeboSystem</plugin>
       </hardware>
-      <!-- <joint name="joint_body">
+      <joint name="joint_body">
         <command_interface name="position">
           <param name="min">0.0</param>
@@ -17,5 +17,5 @@
         <state_interface name="velocity"/>
         <state_interface name="effort"/>
-      </joint> -->
+      </joint>
       <joint name="joint_wheel">
         <command_interface name="effort"/>
