Commit message: Revert "Merge pull request #4 from TanawatPawanta/NutGoingToJump"
This reverts commit d31b15310b6ab68b4e76366a8853ed90fc889992, reversing
changes made to dd2120c0914e55e31adda59f8da0665b5becb546.

File: balegce_gazebo/robot/balegce_sensor.gazebo.xacro (robot description, xacro)
@@ -65,4 +65,20 @@
             </sensor>
         </gazebo>
+        <!-- floor contact -->
+        <gazebo reference="leg">
+            <sensor name="contact_sensor" type="contact">
+                <always_on>true</always_on>
+                <update_rate>10.0</update_rate>
+                <contact>
+                    <collision>leg_collision</collision>
+                </contact>
+                <plugin name="contact_plugin" filename="libgazebo_ros_bumper.so">
+                    <ros>
+                        <remapping>bumper_states:=contact</remapping>
+                    </ros>
+                    <frame_name>leg</frame_name>
+                </plugin>
+            </sensor>
+        </gazebo>
     </xacro:macro>
 </robot>
