Commit message: successfully lift the robot by itself using effort controller

File: balegce/robot/visual/functions.xacro (robot description, xacro)
@@ -1,9 +1,9 @@
 <?xml version='1.0' encoding='utf-8'?>
 <robot xmlns:xacro="http://www.ros.org/wiki/xacro">
-    <xacro:macro name="worldPlan" params=" size xyz rpy">
+    <xacro:macro name="worldPlan" params="mass origin rpy x y z">
         <visual>
-            <origin xyz="${xyz}" rpy="${rpy}"/>
+            <origin xyz="${origin}" rpy="${rpy}"/>
             <geometry>
-                <box size="${size}"/>
+                <box size="${x} ${y} ${z}"/>
             </geometry>
             <material name="worldPlan">
@@ -11,8 +11,24 @@
             </material>
         </visual>
+        <inertial>
+            <origin xyz="${origin}"/>
+            <mass value= "${mass}"/>
+            <inertia ixx="${(1/12) * mass * (y*y+z*z)}"
+                     ixy="0.0"
+                     ixz="0.0"
+                     iyy="${(1/12) * mass * (x*x+z*z)}"
+                     iyz="0.0"
+                     izz="${(1/12) * mass * (x*x+y*y)}" />
+        </inertial>
+        <collision>
+            <origin xyz="${origin}" rpy="${rpy}"/>
+            <geometry>
+                <box size="${x} ${y} ${z}"/>
+            </geometry>
+        </collision>
     </xacro:macro>
-    <xacro:macro name="base_visual" params="xyz rpy R l">
+    <xacro:macro name="base_visual" params="mass origin rpy R l">
         <visual>
-            <origin xyz="${xyz}" rpy="${rpy}"/>
+            <origin xyz="${origin}" rpy="${rpy}"/>
             <geometry>
                 <cylinder radius="${R}" length="${l}"/>
@@ -22,8 +38,24 @@
             </material>
         </visual>
+        <inertial>
+            <origin xyz="${origin}"/>
+            <mass value="${mass}" />
+            <inertia ixx="${(1/12) * mass * (3*R*R + l*l)}"
+                     ixy="0.0"
+                     ixz="0.0"
+                     iyy="${(1/12) * mass * (3*R*R + l*l)}"
+                     iyz="0.0"
+                     izz="${(1/2) * mass * (R*R)}" />
+        </inertial>
+        <collision>
+            <origin xyz="${origin}" rpy="${rpy}"/>
+            <geometry>
+                <cylinder radius="${R}" length="${l}"/>
+            </geometry>
+        </collision>
     </xacro:macro>
-    <xacro:macro name="cylinderSolid" params="link_id xyz rpy R l">
+    <xacro:macro name="cylinderSolid" params="mass origin rpy R l link_id">
         <visual>
-            <origin xyz="${xyz}" rpy="${rpy}"/>
+            <origin xyz="${origin}" rpy="${rpy}"/>
             <geometry>
                 <cylinder radius="${R}" length="${l}"/>
@@ -33,10 +65,26 @@
             </material>
         </visual>
+        <inertial>
+            <origin xyz="${origin}"/>
+            <mass value="${mass}" />
+            <inertia ixx="${(1/12) * mass * (3*R*R + l*l)}"
+                     ixy="0.0"
+                     ixz="0.0"
+                     iyy="${(1/12) * mass * (3*R*R + l*l)}"
+                     iyz="0.0"
+                     izz="${(1/2) * mass * (R*R)}" />
+        </inertial>
+        <collision>
+            <origin xyz="${origin}" rpy="${rpy}"/>
+            <geometry>
+                <cylinder radius="${R}" length="${l}"/>
+            </geometry>
+        </collision>
     </xacro:macro>
-    <xacro:macro name="brickSolid" params="link_id size xyz rpy">
+    <xacro:macro name="brickSolid" params="mass origin rpy x y z link_id">
         <visual>
-            <origin xyz="${xyz}" rpy="${rpy}"/>
+            <origin xyz="${origin}" rpy="${rpy}"/>
             <geometry>
-                <box size="${size}"/>
+                <box size="${x} ${y} ${z}"/>
             </geometry>
             <material name="link_color_${link_id}">
@@ -44,15 +92,31 @@
             </material>
         </visual>
+        <inertial>
+            <origin xyz="${origin}"/>
+            <mass value= "${mass}"/>
+            <inertia ixx="${(1/12) * mass * (y*y+z*z)}"
+                     ixy="0.0"
+                     ixz="0.0"
+                     iyy="${(1/12) * mass * (x*x+z*z)}"
+                     iyz="0.0"
+                     izz="${(1/12) * mass * (x*x+y*y)}" />
+        </inertial>
+        <collision>
+            <origin xyz="${origin}" rpy="${rpy}"/>
+            <geometry>
+                <box size="${x} ${y} ${z}"/>
+            </geometry>
+        </collision>
     </xacro:macro>
-    <xacro:macro name="rigidTransform" params="curr_link next_link xyz rpy">
+    <xacro:macro name="rigidTransform" params="curr_link next_link origin rpy">
         <joint name="rigidTransform_${curr_link}_to_${next_link}" type="fixed">
-            <origin xyz="${xyz}" rpy="${rpy}"/>
+            <origin xyz="${origin}" rpy="${rpy}"/>
             <parent link="${curr_link}"/>
             <child link="${next_link}"/>
         </joint>
     </xacro:macro>
-    <xacro:macro name="revoluteJoint" params="id curr_link next_link xyz rpy">
+    <xacro:macro name="revoluteJoint" params="id curr_link next_link origin rpy">
         <joint name="revoluteJoint_${id}" type="revolute">
-            <origin xyz="${xyz}" rpy="${rpy}"/>
+            <origin xyz="${origin}" rpy="${rpy}"/>
             <parent link="${curr_link}"/>
             <child link="${next_link}"/>
@@ -65,7 +129,7 @@
         </joint>
     </xacro:macro>
-    <xacro:macro name="prismaticJoint" params="id curr_link next_link xyz rpy">
+    <xacro:macro name="prismaticJoint" params="id curr_link next_link origin rpy">
         <joint name="prismaticJoint_${id}" type="prismatic">
-            <origin xyz="${xyz}" rpy="${rpy}"/>
+            <origin xyz="${origin}" rpy="${rpy}"/>
             <parent link="${curr_link}"/>
             <child link="${next_link}"/>

File: balegce/robot/visual/prismatic_1dof.xacro (robot description, xacro)
@@ -7,16 +7,20 @@
     <xacro:include filename="$(find ${package_name})/robot/visual/functions.xacro"/>
     <!-- 1 DOF prismatic -->
-    <link name="world"/>
-    <xacro:rigidTransform curr_link="world" next_link="worldPlan" xyz="0 0 0.05" rpy="0 0 0"/>
+    <!-- <link name="world"/> -->
+    <!-- <xacro:rigidTransform curr_link="world" next_link="worldPlan" origin="0 0 0.05" rpy="0 0 0"/>
     <link name="worldPlan">
-       <xacro:worldPlan  size="5.0 5.0 0.1" xyz="0 0 0" rpy="0 0 0"/>
+       <xacro:worldPlan mass = "10.0" origin="0 0 0" rpy="0 0 0" x="5.0" y="5.0" z="0.1"/>
+    </link> -->
+    <!-- <xacro:rigidTransform curr_link="world" next_link="link_0" origin="0 0 0.10" rpy="0 0 0"/> -->
+    <link name="link_0">
+        <xacro:brickSolid mass = "1.0" origin="0 0 0" rpy="0 0 0" x="0.5" y="0.2" z="0.2" link_id="0"/>
     </link>
-    <xacro:rigidTransform curr_link="worldPlan" next_link="link_0" xyz="0 0 0.15" rpy="0 0 0"/>
-    <link name="link_0">
-        <xacro:brickSolid link_id="0" size="0.5 0.2 0.2" xyz="0 0 0" rpy="0 0 0"/>
+    <xacro:prismaticJoint id="0" curr_link="link_0" next_link="link_1" origin="0.25 0 0.15" rpy="0 ${PI/2} 0"/>
+    <link name="link_1">
+        <xacro:cylinderSolid mass = "1.0" origin="0 0 0" rpy="0 0 0" R="0.05" l="1.0" link_id="1"/>
     </link>
-    <xacro:prismaticJoint id="0" curr_link="link_0" next_link="link_1" xyz="0.5 0 0.15" rpy="0 ${PI/2} 0"/>
-    <link name="link_1">
-        <xacro:cylinderSolid link_id="1" R="0.05" l="1.0" xyz="0 0 0" rpy="0 0 0"/>
+    <xacro:rigidTransform curr_link="link_0" next_link="link_2" origin="0 0 0.30" rpy="0 0 0"/>
+    <link name="link_2">
+        <xacro:brickSolid mass = "1.0" origin="0 0 0" rpy="0 0 0" x="0.5" y="0.2" z="0.2" link_id="2"/>
     </link>
 </robot>

File: balegce_gazebo/robot/balegce.gazebo.xacro (robot description, xacro)
@@ -7,9 +7,9 @@
     <!-- Include sensor plugin -->
     <xacro:include filename="$(find ${gazebo_pkg})/robot/balegce_sensor.gazebo.xacro"/>
+    <!-- Include controller plugin -->
     <xacro:include filename="$(find ${gazebo_pkg})/robot/balegce_controller.gazebo.xacro"/>
     <!-- Add manipulator -->
     <xacro:include filename="$(find ${description_pkg})/robot/visual/manipulator.xacro"/>
-    <xacro:include filename="$(find ${description_package})/robot/visual/sensor.xacro"/>
-    <!-- <link name="world"/> -->
+    <xacro:include filename="$(find ${description_pkg})/robot/visual/sensor.xacro"/>
     <xacro:balegce/>
     <xacro:sensor_link/>

File: balegce_gazebo/robot/balegce_controller.gazebo.xacro (robot description, xacro)
@@ -8,10 +8,5 @@
       </hardware>
       <joint name="joint_body">
-        <command_interface name="position">
-          <param name="min">0.0</param>
-          <param name="max">0.065</param>
-        </command_interface>
         <command_interface name="effort"/>
-        <command_interface name="velocity"/>
         <state_interface name="position"/>
         <state_interface name="velocity"/>
@@ -19,5 +14,4 @@
       </joint>
       <joint name="joint_wheel">
-        <command_interface name="effort"/>
         <command_interface name="velocity"/>
         <state_interface name="position"/>
@@ -26,5 +20,4 @@
       </joint>
       <joint name="joint_propeller_1">
-        <command_interface name="effort"/>
         <command_interface name="velocity"/>
         <state_interface name="position"/>
@@ -33,5 +26,4 @@
       </joint>
       <joint name="joint_propeller_2">
-        <command_interface name="effort"/>
         <command_interface name="velocity"/>
         <state_interface name="position"/>
