Commit message: add contact sensor frame, joint state pub, all joints velocity controller

File: balegce/robot/visual/manipulator.xacro (robot description, xacro)
@@ -231,4 +231,10 @@
             <xacro:propeller_2_collision />
         </link>
+        <link name="end_leg"/>
+        <joint name="joint_end_leg" type="fixed">
+            <parent link="leg"/>
+            <child link="end_leg"/>
+            <origin xyz="0.0 0.0 -0.145" rpy="0.0 0.0 0.0"/>
+        </joint>
         <xacro:base_offset/>
         <xacro:joint_body/>

File: balegce/robot/visual/sensor.xacro (robot description, xacro)
@@ -8,4 +8,10 @@
             <origin xyz="${SENSOR['imu']['position']}" rpy="${SENSOR['imu']['orientation']}"/>
         </joint>
+        <link name="contact_link"/>
+        <joint name="contact_offset" type="fixed">
+            <parent link="${SENSOR['contact']['link']}"/>
+            <child link="contact_link"/>
+            <origin xyz="${SENSOR['contact']['position']}" rpy="${SENSOR['contact']['orientation']}"/>
+        </joint>
     </xacro:macro>
 </robot>

File: balegce_gazebo/robot/balegce_controller.gazebo.xacro (robot description, xacro)
@@ -7,5 +7,26 @@
         <plugin>gazebo_ros2_control/GazeboSystem</plugin>
       </hardware>
+      <joint name="joint_body">
+        <command_interface name="effort"/>
+        <command_interface name="velocity"/>
+        <state_interface name="position"/>
+        <state_interface name="velocity"/>
+        <state_interface name="effort"/>
+      </joint>
       <joint name="joint_wheel">
+        <command_interface name="effort"/>
+        <command_interface name="velocity"/>
+        <state_interface name="position"/>
+        <state_interface name="velocity"/>
+        <state_interface name="effort"/>
+      </joint>
+      <joint name="joint_propeller_1">
+        <command_interface name="effort"/>
+        <command_interface name="velocity"/>
+        <state_interface name="position"/>
+        <state_interface name="velocity"/>
+        <state_interface name="effort"/>
+      </joint>
+      <joint name="joint_propeller_2">
         <command_interface name="effort"/>
         <command_interface name="velocity"/>

Commit message: 2 Propeller force generate

File: balegce/robot/visual/manipulator.xacro (robot description, xacro)
@@ -27,5 +27,5 @@
     <xacro:macro name="leg_collision">
         <collision>
-            <origin xyz="${LEG_COLLISION['position']}" rpy="${LEG_COLLISION['orientation']}"/>
+            <origin xyz="${LEG_VISUAL['position']}" rpy="${LEG_VISUAL['orientation']}"/>
             <geometry>
                 <mesh filename="file://$(find ${description_package})/meshes/leg.stl"/>
@@ -59,5 +59,5 @@
     <xacro:macro name="body_collision">
         <collision>
-            <origin xyz="${BODY_COLLISION['position']}" rpy="${BODY_COLLISION['orientation']}"/>
+            <origin xyz="${BODY_VISUAL['position']}" rpy="${BODY_VISUAL['orientation']}"/>
             <geometry>
                 <mesh filename="file://$(find ${description_package})/meshes/body.stl"/>
@@ -91,5 +91,5 @@
     <xacro:macro name="reactionwheel_collision">
         <collision>
-            <origin xyz="${REACTIONWHEEL_COLLISION['position']}" rpy="${REACTIONWHEEL_COLLISION['orientation']}"/>
+            <origin xyz="${REACTIONWHEEL_VISUAL['position']}" rpy="${REACTIONWHEEL_VISUAL['orientation']}"/>
             <geometry>
                 <mesh filename="file://$(find ${description_package})/meshes/reactionwheel.stl"/>
@@ -134,5 +134,5 @@
     <xacro:macro name="propeller_1_collision">
         <collision>
-            <origin xyz="${PROPELLER_COLLISION['position']}" rpy="${PROPELLER_COLLISION['orientation']}"/>
+            <origin xyz="${PROPELLER_1_VISUAL['position']}" rpy="${PROPELLER_1_VISUAL['orientation']}"/>
             <geometry>
                 <mesh filename="file://$(find ${description_package})/meshes/propeller_1.stl"/>
@@ -142,5 +142,5 @@
     <xacro:macro name="propeller_2_collision">
         <collision>
-            <origin xyz="${PROPELLER_COLLISION['position']}" rpy="${PROPELLER_COLLISION['orientation']}"/>
+            <origin xyz="${PROPELLER_2_VISUAL['position']}" rpy="${PROPELLER_2_VISUAL['orientation']}"/>
             <geometry>
                 <mesh filename="file://$(find ${description_package})/meshes/propeller_2.stl"/>

File: balegce/robot/visual/robot.xacro (robot description, xacro)
@@ -10,5 +10,5 @@
     <xacro:include filename="$(find ${description_package})/robot/visual/sensor.xacro"/>
     <xacro:balegce/>
-    <!-- attrach sensor -->
+    <!-- attach sensor -->
     <xacro:sensor_link/>
 </robot>

File: balegce_gazebo/robot/balegce.gazebo.xacro (robot description, xacro)
@@ -7,4 +7,5 @@
     <!-- Include sensor plugin -->
     <xacro:include filename="$(find ${gazebo_pkg})/robot/balegce_sensor.gazebo.xacro"/>
+    <!-- Include controller plugin -->
     <xacro:include filename="$(find ${gazebo_pkg})/robot/balegce_controller.gazebo.xacro"/>
     <!-- Add manipulator -->
@@ -21,4 +22,4 @@
     <xacro:sensor_link/>
     <xacro:sensor_plugins/>
-    <xacro:velocity_controller/>
+    <xacro:controller/>
 </robot>

File: balegce_gazebo/robot/balegce_controller.gazebo.xacro (robot description, xacro)
@@ -1,5 +1,5 @@
 <?xml version='1.0' encoding='utf-8'?>
 <robot xmlns:xacro="http://www.ros.org/wiki/xacro">
-  <xacro:macro name="velocity_controller" params="">
+  <xacro:macro name="controller" params="">
     <xacro:property name="controller_file" value="controller_config.yaml"/>
     <ros2_control name="GazeboSystem" type="system">
@@ -8,6 +8,14 @@
       </hardware>
       <joint name="joint_wheel">
+        <command_interface name="velocity"/>
         <command_interface name="effort"/>
+        <state_interface name="position"/>
+        <state_interface name="velocity"/>
+        <state_interface name="effort"/>
+      </joint>
+      <joint name="leg">
+        <command_interface name="position"/>
         <command_interface name="velocity"/>
+        <command_interface name="effort"/>
         <state_interface name="position"/>
         <state_interface name="velocity"/>
@@ -20,4 +28,32 @@
       </plugin>
     </gazebo>
+    <gazebo>
+      <plugin filename="libgazebo_ros_force.so" name="gazebo_ros_force">
+      <ros>
+        <namespace>/propeller_r</namespace>
+        <remapping>gazebo_ros_force:=force</remapping>
+      </ros>
+          <alwaysOn>true</alwaysOn>
+          <update>100</update>
+          <updateRate>100.0</updateRate>
+          <link_name>propeller_1</link_name>
+          <force_frame>link</force_frame>
+          <enableCommand>true</enableCommand>
+      </plugin>
+    </gazebo>
+    <gazebo>
+      <plugin filename="libgazebo_ros_force.so" name="gazebo_ros_force">
+      <ros>
+        <namespace>/propeller_l</namespace>
+        <remapping>gazebo_ros_force:=force</remapping>
+      </ros>
+          <alwaysOn>true</alwaysOn>
+          <update>100</update>
+          <updateRate>100.0</updateRate>
+          <link_name>propeller_2</link_name>
+          <force_frame>link</force_frame>
+          <enableCommand>true</enableCommand>
+      </plugin>
+    </gazebo>
   </xacro:macro>
 </robot>

Commit message: change leg to prismatic, add mu to leg

File: balegce/robot/visual/manipulator.xacro (robot description, xacro)
@@ -205,4 +205,5 @@
     <!-- Visual with dynamics propoties -->
     <xacro:macro name="balegce" params="">
+        <link name="end_leg"/>
         <link name="base"/>
         <link name="leg">
@@ -231,5 +232,4 @@
             <xacro:propeller_2_collision />
         </link>
-        <link name="end_leg"/>
         <joint name="joint_end_leg" type="fixed">
             <parent link="leg"/>

File: balegce_gazebo/robot/balegce_controller.gazebo.xacro (robot description, xacro)
@@ -70,3 +70,8 @@
       </plugin>
     </gazebo>
+    <gazebo reference="leg">
+        <mu1>0.2</mu1>
+        <mu2>0.2</mu2>
+        <material>Gazebo/Green</material>
+    </gazebo>
 </robot>

Commit message: Model Correction

File: balegce/robot/visual/manipulator.xacro (robot description, xacro)
@@ -27,5 +27,5 @@
     <xacro:macro name="leg_collision">
         <collision>
-            <origin xyz="${LEG_COLLISION['position']}" rpy="${LEG_COLLISION['orientation']}"/>
+            <origin xyz="${LEG_VISUAL['position']}" rpy="${LEG_VISUAL['orientation']}"/>
             <geometry>
                 <mesh filename="file://$(find ${description_package})/meshes/leg.stl"/>
@@ -59,5 +59,5 @@
     <xacro:macro name="body_collision">
         <collision>
-            <origin xyz="${BODY_COLLISION['position']}" rpy="${BODY_COLLISION['orientation']}"/>
+            <origin xyz="${BODY_VISUAL['position']}" rpy="${BODY_VISUAL['orientation']}"/>
             <geometry>
                 <mesh filename="file://$(find ${description_package})/meshes/body.stl"/>
@@ -91,5 +91,5 @@
     <xacro:macro name="reactionwheel_collision">
         <collision>
-            <origin xyz="${REACTIONWHEEL_COLLISION['position']}" rpy="${REACTIONWHEEL_COLLISION['orientation']}"/>
+            <origin xyz="${REACTIONWHEEL_VISUAL['position']}" rpy="${REACTIONWHEEL_VISUAL['orientation']}"/>
             <geometry>
                 <mesh filename="file://$(find ${description_package})/meshes/reactionwheel.stl"/>
@@ -134,5 +134,5 @@
     <xacro:macro name="propeller_1_collision">
         <collision>
-            <origin xyz="${PROPELLER_COLLISION['position']}" rpy="${PROPELLER_COLLISION['orientation']}"/>
+            <origin xyz="${PROPELLER_1_VISUAL['position']}" rpy="${PROPELLER_1_VISUAL['orientation']}"/>
             <geometry>
                 <mesh filename="file://$(find ${description_package})/meshes/propeller_1.stl"/>
@@ -142,5 +142,5 @@
     <xacro:macro name="propeller_2_collision">
         <collision>
-            <origin xyz="${PROPELLER_COLLISION['position']}" rpy="${PROPELLER_COLLISION['orientation']}"/>
+            <origin xyz="${PROPELLER_2_VISUAL['position']}" rpy="${PROPELLER_2_VISUAL['orientation']}"/>
             <geometry>
                 <mesh filename="file://$(find ${description_package})/meshes/propeller_2.stl"/>

Commit message: add to gazebo

File: balegce/robot/visual/manipulator.xacro (robot description, xacro)
@@ -157,6 +157,6 @@
     <xacro:macro name="joint_body" params="">
         <joint name="joint_body" type="${JOINT_BODY['types']}">
-            <parent link="body"/>
-            <child link="leg"/>
+            <parent link="leg"/>
+            <child link="body"/>
             <origin xyz="${JOINT_BODY['position']}" rpy="${JOINT_BODY['orientation']}"/>
             <axis xyz="0 0 1"/>
@@ -203,8 +203,40 @@
         </joint>
     </xacro:macro>
+    <xacro:macro name="rigidTransform" params="curr_link next_link xyz rpy">
+        <joint name="rigidTransform_${curr_link}_to_${next_link}" type="fixed">
+            <origin xyz="${xyz}" rpy="${rpy}"/>
+            <parent link="${curr_link}"/>
+            <child link="${next_link}"/>
+        </joint>
+    </xacro:macro>
+    <xacro:macro name="revoluteJoint" params="id curr_link next_link xyz rpy">
+        <joint name="revoluteJoint_${id}" type="revolute">
+            <origin xyz="${xyz}" rpy="${rpy}"/>
+            <parent link="${curr_link}"/>
+            <child link="${next_link}"/>
+            <axis xyz="0 0 1"/>
+            <limit
+                lower="-3.14152"
+                upper="3.14152"
+                velocity="1000.0"
+                effort="1000.0"/>
+        </joint>
+    </xacro:macro>
     <!-- Visual with dynamics propoties -->
+    <xacro:property name="PI" value="3.141592653589793"/>
     <xacro:macro name="balegce" params="">
-        <link name="end_leg"/>
-        <link name="base"/>
+        <link name="world"/>
+        <joint name="revoluteJoint_0" type="revolute">
+                <origin xyz="0 0 0" rpy="0 0 0"/>
+                <parent link="world"/>
+                <child link="leg"/>
+                <axis xyz="1 0 0"/>
+                <limit
+                    lower="-${PI/2}"
+                    upper="${PI/2}"
+                    velocity="1000.0"
+                    effort="1000.0"/>
+        </joint>
+        <!-- <link name="base"/> -->
         <link name="leg">
             <xacro:leg_visual />
@@ -232,10 +264,5 @@
             <xacro:propeller_2_collision />
         </link>
-        <joint name="joint_end_leg" type="fixed">
-            <parent link="leg"/>
-            <child link="end_leg"/>
-            <origin xyz="0.0 0.0 -0.145" rpy="0.0 0.0 0.0"/>
-        </joint>
-        <xacro:base_offset/>
+        <!-- <xacro:base_offset/> -->
         <xacro:joint_body/>
         <xacro:joint_wheel/>

File: balegce/robot/visual/robot.xacro (robot description, xacro)
@@ -9,4 +9,17 @@
     <xacro:include filename="$(find ${description_package})/robot/visual/manipulator.xacro"/>
     <xacro:include filename="$(find ${description_package})/robot/visual/sensor.xacro"/>
+    <xacro:property name="PI" value="3.141592653589793"/>
+    <link name="world"/>
+    <joint name="revoluteJoint_0" type="revolute">
+            <origin xyz="0 0 0" rpy="0 0 0"/>
+            <parent link="world"/>
+            <child link="leg"/>
+            <axis xyz="1 0 0"/>
+            <limit
+                lower="-$(PI/2)"
+                upper="$(PI/2)"
+                velocity="1000.0"
+                effort="1000.0"/>
+    </joint>
     <xacro:balegce/>
     <!-- attrach sensor -->

Commit message: Contact sensor (Completed)
https://answers.gazebosim.org//question/15095/gazebo-contact-sensor-added-to-a-robot-link-in-urdf-file-is-not-working-as-expected/

File: balegce/robot/visual/manipulator.xacro (robot description, xacro)
@@ -26,5 +26,5 @@
     </xacro:macro>
     <xacro:macro name="leg_collision">
-        <collision>
+        <collision name="leg_collision">
             <origin xyz="${LEG_VISUAL['position']}" rpy="${LEG_VISUAL['orientation']}"/>
             <geometry>

File: balegce_gazebo/robot/balegce_sensor.gazebo.xacro (robot description, xacro)
@@ -66,18 +66,16 @@
         </gazebo>
         <!-- floor contact -->
-        <gazebo reference="contact_link">
-            <gravity>true</gravity>
+        <gazebo reference="leg">
             <sensor name="contact_sensor" type="contact">
                 <always_on>true</always_on>
-                <update_rate>10</update_rate>
-                <visualize>true</visualize>
-                <topic>__default_topic__</topic>
-                <plugin filename="libgazebo_ros_contact.so" name="contact_plugin">
+                <update_rate>10.0</update_rate>
+                <contact>
+                    <collision>leg_collision_collision</collision>
+                </contact>
+                <plugin name="contact_plugin" filename="libgazebo_ros_bumper.so">
                     <ros>
-                        <remapping>~/out:=contact</remapping>
+                        <remapping>bumper_states:=contact</remapping>
                     </ros>
-                    <update_rate>10.0</update_rate>
-                    <gaussian_noise>0.0</gaussian_noise>
-                    <frame_name>contact_link</frame_name>
+                    <frame_name>leg</frame_name>
                 </plugin>
             </sensor>

Commit message: minor

File: balegce/robot/visual/manipulator.xacro (robot description, xacro)
@@ -26,5 +26,5 @@
     </xacro:macro>
     <xacro:macro name="leg_collision">
-        <collision name="leg_collision">
+        <collision name="leg">
             <origin xyz="${LEG_VISUAL['position']}" rpy="${LEG_VISUAL['orientation']}"/>
             <geometry>

File: balegce_gazebo/robot/balegce_sensor.gazebo.xacro (robot description, xacro)
@@ -71,5 +71,5 @@
                 <update_rate>10.0</update_rate>
                 <contact>
-                    <collision>leg_collision_collision</collision>
+                    <collision>leg_collision</collision>
                 </contact>
                 <plugin name="contact_plugin" filename="libgazebo_ros_bumper.so">

Commit message: minor

File: balegce/robot/visual/manipulator.xacro (robot description, xacro)
@@ -26,9 +26,5 @@
     </xacro:macro>
     <xacro:macro name="leg_collision">
-<<<<<<< HEAD
-        <collision>
-=======
-        <collision name="leg">
->>>>>>> main
+        <collision>
             <origin xyz="${LEG_VISUAL['position']}" rpy="${LEG_VISUAL['orientation']}"/>
             <geometry>
@@ -209,5 +205,4 @@
     <!-- Visual with dynamics propoties -->
     <xacro:macro name="balegce" params="">
-        <link name="end_leg"/>
         <link name="base"/>
         <link name="leg">
@@ -236,9 +231,4 @@
             <xacro:propeller_2_collision />
         </link>
-        <joint name="joint_end_leg" type="fixed">
-            <parent link="leg"/>
-            <child link="end_leg"/>
-            <origin xyz="0.0 0.0 -0.145" rpy="0.0 0.0 0.0"/>
-        </joint>
         <xacro:base_offset/>
         <xacro:joint_body/>

File: balegce/robot/visual/sensor.xacro (robot description, xacro)
@@ -8,10 +8,4 @@
             <origin xyz="${SENSOR['imu']['position']}" rpy="${SENSOR['imu']['orientation']}"/>
         </joint>
-        <link name="contact_link"/>
-        <joint name="contact_offset" type="fixed">
-            <parent link="${SENSOR['contact']['link']}"/>
-            <child link="contact_link"/>
-            <origin xyz="${SENSOR['contact']['position']}" rpy="${SENSOR['contact']['orientation']}"/>
-        </joint>
     </xacro:macro>
 </robot>

File: balegce_gazebo/robot/balegce.gazebo.xacro (robot description, xacro)
@@ -9,5 +9,4 @@
     <!-- Include controller plugin -->
     <xacro:include filename="$(find ${gazebo_pkg})/robot/balegce_controller.gazebo.xacro"/>
-    <xacro:include filename="$(find ${gazebo_pkg})/robot/balegce_ground_truth.xacro"/>
     <!-- Add manipulator -->
     <xacro:include filename="$(find ${description_pkg})/robot/visual/manipulator.xacro"/>
@@ -15,4 +14,10 @@
     <!-- <link name="world"/> -->
     <xacro:balegce/>
+    <!-- <joint name="offset" type="floating">
+        <parent link="world"/>
+        <child link="base"/>
+        <origin xyz="0.0 0.0 0.15" rpy="0.0 0.0 0.0"/>
+        <axis xyz="0 0 1"/>
+    </joint> -->
     <xacro:sensor_link/>
     <xacro:sensor_plugins/>

File: balegce_gazebo/robot/balegce_controller.gazebo.xacro (robot description, xacro)
@@ -7,31 +7,5 @@
         <plugin>gazebo_ros2_control/GazeboSystem</plugin>
       </hardware>
-<<<<<<< HEAD
       <joint name="joint_wheel">
-=======
-      <joint name="joint_body">
-        <command_interface name="position">
-          <param name="min">0.0</param>
-          <param name="max">0.065</param>
-        </command_interface>
-        <command_interface name="effort"/>
-        <state_interface name="position"/>
-        <state_interface name="velocity"/>
-        <state_interface name="effort"/>
-      </joint>
-      <joint name="joint_wheel">
-        <command_interface name="velocity"/>
-        <state_interface name="position"/>
-        <state_interface name="velocity"/>
-        <state_interface name="effort"/>
-      </joint>
-      <joint name="joint_propeller_1">
-        <command_interface name="velocity"/>
-        <state_interface name="position"/>
-        <state_interface name="velocity"/>
-        <state_interface name="effort"/>
-      </joint>
-      <joint name="joint_propeller_2">
->>>>>>> main
         <command_interface name="velocity"/>
         <command_interface name="effort"/>
@@ -83,36 +57,3 @@
     </gazebo>
   </xacro:macro>
-      <gazebo>
-      <plugin filename="libgazebo_ros_force.so" name="gazebo_ros_force">
-      <ros>
-        <namespace>/propeller_r</namespace>
-        <remapping>gazebo_ros_force:=force</remapping>
-      </ros>
-          <alwaysOn>true</alwaysOn>
-          <update>100</update>
-          <updateRate>100.0</updateRate>
-          <link_name>propeller_1</link_name>
-          <force_frame>link</force_frame>
-          <enableCommand>true</enableCommand>
-      </plugin>
-    </gazebo>
-    <gazebo>
-      <plugin filename="libgazebo_ros_force.so" name="gazebo_ros_force">
-      <ros>
-        <namespace>/propeller_l</namespace>
-        <remapping>gazebo_ros_force:=force</remapping>
-      </ros>
-          <alwaysOn>true</alwaysOn>
-          <update>100</update>
-          <updateRate>100.0</updateRate>
-          <link_name>propeller_2</link_name>
-          <force_frame>link</force_frame>
-          <enableCommand>true</enableCommand>
-      </plugin>
-    </gazebo>
-    <gazebo reference="leg">
-        <mu1>0.2</mu1>
-        <mu2>0.2</mu2>
-        <material>Gazebo/Green</material>
-    </gazebo>
 </robot>

File: balegce_gazebo/robot/balegce_sensor.gazebo.xacro (robot description, xacro)
@@ -65,20 +65,4 @@
             </sensor>
         </gazebo>
-        <!-- floor contact -->
-        <gazebo reference="leg">
-            <sensor name="contact_sensor" type="contact">
-                <always_on>true</always_on>
-                <update_rate>10.0</update_rate>
-                <contact>
-                    <collision>leg_collision</collision>
-                </contact>
-                <plugin name="contact_plugin" filename="libgazebo_ros_bumper.so">
-                    <ros>
-                        <remapping>bumper_states:=contact</remapping>
-                    </ros>
-                    <frame_name>leg</frame_name>
-                </plugin>
-            </sensor>
-        </gazebo>
     </xacro:macro>
 </robot>
